File: Juice Rescue v2 - KICAD/Juice Rescue v2 - hw1.0.2/Juice Rescue v2 - hw1.0.2.kicad_sch (KiCad schematic)
At the start: 144 parts, among them IC1 LMV358, IC2 ATMEGA328P-AU, IC3 LM358, IC4 TC1044S, IC5 MCP23017SO, IC7 AQH2223, IC8 HCPL-2731S, J1 CONN_02, M1 MOV, M2 MOV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

Commit message: level shifter and temp
Parts:
- removed D13: 1N4148, Juice Rescue v2 - hw1.0.2:SOD123, symbol Juice Rescue v2 - hw1.0.2-eagle-import:DIODE-SOD123
- added C38: 1.0uF, Juice Rescue v2 - hw1.0.2:0805, symbol Juice Rescue v2 - hw1.0.2-eagle-import:1.0UF-0805-25V-(+80/-20%)
- added JP1: EX_A0, symbol Jumper:Jumper_2_Small_Bridged
- added JP2: EX_A1, symbol Jumper:Jumper_2_Small_Bridged
- added JP3: EX_A2, symbol Jumper:Jumper_2_Small_Bridged
- added JP4: MCP1_A0, symbol Jumper:Jumper_2_Small_Bridged
- added JP5: MCP1_A1, symbol Jumper:Jumper_2_Small_Bridged
- added JP6: MCP1_A2, symbol Jumper:Jumper_2_Small_Bridged
- added JP7: MCP0_A0, symbol Jumper:Jumper_2_Small_Bridged
- added JP8: MCP0_A1, symbol Jumper:Jumper_2_Small_Bridged
- added JP9: MCP0_A2, symbol Jumper:Jumper_2_Small_Bridged
- added Q3, Q4: BSS138, Package_TO_SOT_SMD:SOT-23, symbol Transistor_FET:BSS138
- added R40, R41, R42, R43: 10K, PCM_JLCPCB:R_0805, symbol Device:R
- added R44, R45: 4.7k, Juice Rescue v2 - hw1.0.2:0805, symbol Juice Rescue v2 - hw1.0.2-eagle-import:RESISTOR0805-RES
- added TP1: RXD0, TestPoint:TestPoint_Pad_D2.0mm, symbol Connector:TestPoint
- added TP2: TXD0, TestPoint:TestPoint_Pad_D2.0mm, symbol Connector:TestPoint
- added TP3: TX1, TestPoint:TestPoint_Pad_D2.0mm, symbol Connector:TestPoint
- added TP4: RX1, TestPoint:TestPoint_Pad_D2.0mm, symbol Connector:TestPoint
- added U3, U4: MCP9808_MSOP, Package_SO:MSOP-8_3x3mm_P0.65mm, symbol Sensor_Temperature:MCP9808_MSOP
- U1: value AP63203 -> AP63205
Connections:
- net +5V: now also R41.1, R43.1, U4.8 (V_{DD})
- net 3.3V: now also Q3.1 (G), Q4.1 (G), R40.1, R42.1, R44.2, R45.2, U3.8 (V_{DD})
- net ESPSCL: now also R45.1, U3.2 (SCL)
- net ESPSDA: now also R44.1, U3.1 (SDA)
- net GND: now also C38.2, JP1.1 (A), JP2.1 (A), JP3.1 (A), JP4.1 (A), JP5.1 (A), JP6.1 (A), JP7.1 (A), JP8.1 (A), JP9.1 (A), U3.4 (GND), U4.4 (GND); no longer IC5.15 (A0), IC5.16 (A1), IC5.17 (A2)
- net GPIO0: now also C38.1
- net RXD0: now also Q4.2 (S), R42.2, TP1.1
- net SCL: now also U4.2 (SCL)
- net SDA: now also U4.1 (SDA)
- net RX-I renamed RX1
- net RX1: now also Q3.3 (D), R41.2, TP4.1; no longer X2.35 (TXD0)
- net TX renamed TX1
- net TX1: now also Q4.3 (D), R43.2, TP3.1
- new net: JP6.2 (B), U4.5 (A2)
- new net: IC5.15 (A0), JP1.2 (B)
- new net: IC5.16 (A1), JP2.2 (B)
- new net: IC5.17 (A2), JP3.2 (B)
- new net: JP4.2 (B), U4.7 (A0)
- new net: JP7.2 (B), U3.7 (A0)
- new net: JP5.2 (B), U4.6 (A1)
- new net: JP8.2 (B), U3.6 (A1)
- new net: JP9.2 (B), U3.5 (A2)
- new net TXD0: Q3.2 (S), R40.2, TP2.1, X2.35 (TXD0)
Other:
- moved on the sheet: C8, R13, RESET0, SFQ0

Commit message: ESP32 update.
Parts:
- removed BOOT0, RESET0: KMR2, Juice Rescue v2 - hw1.0.2:BTN_KMR2_4.6X2.8, symbol Juice Rescue v2 - hw1.0.2-eagle-import:SWITCH_TACT_SMT4.6X2.8
- removed C38, C8: 1.0uF, Juice Rescue v2 - hw1.0.2:0805, symbol Juice Rescue v2 - hw1.0.2-eagle-import:1.0UF-0805-25V-(+80/-20%)
- removed JP7: MCP0_A0, symbol Jumper:Jumper_2_Small_Bridged
- removed JP8: MCP0_A1, symbol Jumper:Jumper_2_Small_Bridged
- removed JP9: MCP0_A2, symbol Jumper:Jumper_2_Small_Bridged
- removed LED0: 3-PIN SMD, Juice Rescue v2 - hw1.0.2:JST-3-SMD, symbol Juice Rescue v2 - hw1.0.2-eagle-import:M03JST-SMD
- removed LED1, LED2: WS2812B3535, Juice Rescue v2 - hw1.0.2:LED3535, symbol Juice Rescue v2 - hw1.0.2-eagle-import:WS2812B3535
- removed Q3, Q4: BSS138, Package_TO_SOT_SMD:SOT-23, symbol Transistor_FET:BSS138
- removed R13: 10k, Juice Rescue v2 - hw1.0.2:0805, symbol Juice Rescue v2 - hw1.0.2-eagle-import:RESISTOR0805
- removed R40, R41, R42, R43: 10K, PCM_JLCPCB:R_0805, symbol Device:R
- removed R44, R45: 4.7k, Juice Rescue v2 - hw1.0.2:0805, symbol Juice Rescue v2 - hw1.0.2-eagle-import:RESISTOR0805-RES
- removed SFQ0: QWIIC_CONNECTORJS-1MM, Juice Rescue v2 - hw1.0.2:JST04_1MM_RA, symbol Juice Rescue v2 - hw1.0.2-eagle-import:QWIIC_CONNECTORJS-1MM
- removed TP1: RXD0, TestPoint:TestPoint_Pad_D2.0mm, symbol Connector:TestPoint
- removed TP2: TXD0, TestPoint:TestPoint_Pad_D2.0mm, symbol Connector:TestPoint
- removed TP3: TX1, TestPoint:TestPoint_Pad_D2.0mm, symbol Connector:TestPoint
- removed TP4: RX1, TestPoint:TestPoint_Pad_D2.0mm, symbol Connector:TestPoint
- removed U3: MCP9808_MSOP, Package_SO:MSOP-8_3x3mm_P0.65mm, symbol Sensor_Temperature:MCP9808_MSOP
- removed X2: ESP32-WROOM-32, Juice Rescue v2 - hw1.0.2:WROOM32_SKINNY, symbol Juice Rescue v2 - hw1.0.2-eagle-import:ESP32_WROOM32_SKINNY
- JP4, JP5, JP6: footprint (none) -> Jumper:SolderJumper-2_P1.3mm_Bridged_RoundedPad1.0x1.5mm
Other:
- added sheet ESP32 (esp32.kicad_sch)
- moved on the sheet: JP4, JP5, JP6, U4
