File: Juice Rescue v2 - KICAD/Juice Rescue v2 - hw1.0.2/Juice Rescue v2 - hw1.0.2.kicad_sch (KiCad schematic)
At the start: 141 parts, among them IC1 LMV358, IC2 ATMEGA328P-AU, IC3 LM358, IC4 TC1044S, IC5 MCP23017SO, IC7 AQH2223, IC8 HCPL-2731S, J1 CONN_02, M1 MOV, M2 MOV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

Commit message: Hw changes.
Connections:
- net +5V: now also U1.1 (FB)
- net 3.3V: now also U2.1 (FB)
- net PP_READ renamed ADC2
- no-connect marks 0 -> 24
