File: Juice Rescue v2 - KICAD/Juice Rescue v2 - hw1.0.2/Juice Rescue v2 - hw1.0.2.kicad_pcb (KiCad board)
At the start: 2 copper layers, 215.8 x 65.1 mm, 148 parts, among them IC1 LMV358, IC2 ATMEGA328P-AU, IC3 LM358, IC4 TC1044S, IC5 MCP23017SO, IC7 AQH2223, IC8 HCPL-2731S, M1 MOV, M2 MOV, M3 MOV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

Commit message: Minor update.
Routing:
- net UGND: track 19.4 -> 18.1 mm
Changed lines of the file:
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@@
 		)
 		(property "Value" "MOV"
-			(at 5.6466 -0.0778 -90)
+			(at 5.6466 -0.0778 270)
 			(unlocked yes)
 			(layer "F.SilkS")
@@
 		)
 		(property "Value" "MOV"
-			(at 4.5274 0.2746 -90)
+			(at 4.5274 0.2746 270)
 			(unlocked yes)
 			(layer "F.SilkS")
@@
 		(descr "MKS3, 10 x 4 mm, grid 7.62 mm")
 		(property "Reference" "C39"
-			(at -9.017 -0.635 -90)
+			(at -9.017 -0.635 270)
 			(unlocked yes)
 			(layer "B.SilkS")
@@
 		)
 		(property "Value" "10000pf"
-			(at -3.81 -3.556 -90)
+			(at -3.81 -3.556 270)
 			(unlocked yes)
 			(layer "B.Fab")
@@
 		(at 184.2581 123.4269 180)
 		(property "Reference" "PS1"
-			(at 1.778 21.59 -0)
+			(at 1.778 21.59 0)
 			(unlocked yes)
 			(layer "B.SilkS")
@@
 		(descr "MKS3, 10 x 4 mm, grid 7.62 mm")
 		(property "Reference" "C40"
-			(at -10.1346 -0.635 -90)
+			(at -10.1346 -0.635 270)
 			(unlocked yes)
 			(layer "B.SilkS")
@@
 		)
 		(property "Value" "10000pf"
-			(at -3.81 -3.556 -90)
+			(at -3.81 -3.556 270)
 			(unlocked yes)
 			(layer "B.Fab")
@@
 	)
 	(segment
-		(start 125.7865 94.1653)
-		(end 125.7619 94.1407)
-		(width 0.3048)
-		(layer "F.Cu")
-		(net 44)
-	)
-	(segment
 		(start 118.4215 93.3653)
 		(end 117.3919 93.3653)
@@
 		(layer "F.Cu")
 		(net 44)
-	)
-	(segment
-		(start 127.0067 94.1653)
-		(end 125.7865 94.1653)
-		(width 0.3048)
-		(layer "F.Cu")
-		(net 44)
